Commit message: feat(sim): migrate to ROS 2 Humble and implement native Ackermann steering

File: urdf/ackerman.xacro (robot description, xacro)
@@ -2,7 +2,5 @@
 <robot name="ack" xmlns:xacro="http://ros.org/wiki/xacro">
   <!-- Materials -->
-  <material name="black">
-    <color rgba="0 0 0 1"/>
-  </material>
+  <xacro:include filename="$(find mentorpia1_simulator)/urdf/materials.xacro" />
   <!-- Base Link -->
   <link name="base_link">
@@ -26,4 +24,7 @@
     </collision>
   </link>
+  <gazebo reference="base_link">
+    <material>Gazebo/Black</material>
+  </gazebo>
   <!-- Base Footprint -->
   <link name="base_footprint"/>
@@ -93,5 +94,10 @@
   </joint>
   <!-- Front Axle and Steering -->
-  <link name="front_axle"/>
+  <link name="front_axle">
+    <inertial>
+      <mass value="0.01"/>
+      <inertia ixx="0.0001" ixy="0" ixz="0" iyy="0.0001" iyz="0" izz="0.0001"/>
+    </inertial>
+  </link>
   <joint name="steering_wheel_joint" type="revolute">
     <parent link="base_link"/>
@@ -101,5 +107,10 @@
     <limit effort="10" velocity="1" lower="-0.4" upper="0.4"/>
   </joint>
-  <link name="left_steering_link"/>
+  <link name="left_steering_link">
+    <inertial>
+      <mass value="0.01"/>
+      <inertia ixx="0.0001" ixy="0" ixz="0" iyy="0.0001" iyz="0" izz="0.0001"/>
+    </inertial>
+  </link>
   <joint name="left_steering_joint" type="revolute">
     <parent link="front_axle"/>
@@ -109,5 +120,10 @@
     <limit effort="10" velocity="1" lower="-0.4" upper="0.4"/>
   </joint>
-  <link name="right_steering_link"/>
+  <link name="right_steering_link">
+    <inertial>
+      <mass value="0.01"/>
+      <inertia ixx="0.0001" ixy="0" ixz="0" iyy="0.0001" iyz="0" izz="0.0001"/>
+    </inertial>
+  </link>
   <joint name="right_steering_joint" type="revolute">
     <parent link="front_axle"/>
@@ -194,6 +210,28 @@
     <parent link="base_link"/>
     <child link="lidar_frame"/>
-    <axis xyz="0 0 0"/>
-  </joint>
+  </joint>
+  <gazebo reference="lidar_frame">
+    <sensor name="gpu_lidar" type="gpu_lidar">
+      <update_rate>10</update_rate>
+      <topic>lidar</topic>
+      <gz_frame_id>lidar_frame</gz_frame_id>
+      <lidar>
+        <scan>
+          <horizontal>
+            <samples>360</samples>
+            <resolution>1</resolution>
+            <min_angle>-3.14159</min_angle>
+            <max_angle>3.14159</max_angle>
+          </horizontal>
+        </scan>
+        <range>
+          <min>0.12</min>
+          <max>12.0</max>
+          <resolution>0.01</resolution>
+        </range>
+      </lidar>
+      <visualize>true</visualize>
+    </sensor>
+  </gazebo>
   <!-- Depth Camera -->
   <link name="depth_cam">
@@ -221,7 +259,59 @@
     <parent link="base_link"/>
     <child link="depth_cam"/>
-    <axis xyz="0 0 0"/>
-  </joint>
+  </joint>
+  <gazebo reference="depth_cam">
+    <sensor name="camera" type="camera">
+      <camera>
+        <horizontal_fov>1.047</horizontal_fov>
+        <image>
+          <width>640</width>
+          <height>480</height>
+        </image>
+        <clip>
+          <near>0.1</near>
+          <far>100</far>
+        </clip>
+      </camera>
+      <always_on>1</always_on>
+      <update_rate>30</update_rate>
+      <visualize>true</visualize>
+      <topic>camera</topic>
+    </sensor>
+  </gazebo>
   <!-- Include IMU -->
   <xacro:include filename="$(find mentorpia1_simulator)/urdf/imu.urdf.xacro"/>
+  <!-- Gazebo Plugins -->
+  <gazebo>
+    <plugin
+      filename="ignition-gazebo-ackermann-steering-system"
+      name="ignition::gazebo::systems::AckermannSteering">
+      <left_joint>wheel_lb_Joint</left_joint>
+      <right_joint>wheel_rb_Joint</right_joint>
+      <steering_joint>steering_wheel_joint</steering_joint>
+      <left_steering_joint>left_steering_joint</left_steering_joint>
+      <right_steering_joint>right_steering_joint</right_steering_joint>
+      <left_rear_wheel_joint>wheel_lb_Joint</left_rear_wheel_joint>
+      <right_rear_wheel_joint>wheel_rb_Joint</right_rear_wheel_joint>
+      <left_front_wheel_joint>wheel_lf_Joint</left_front_wheel_joint>
+      <right_front_wheel_joint>wheel_rf_Joint</right_front_wheel_joint>
+      <wheel_separation>0.14</wheel_separation>
+      <wheelbase>0.14</wheelbase>
+      <wheel_radius>0.035</wheel_radius>
+      <min_steering_angle>-0.4</min_steering_angle>
+      <max_steering_angle>0.4</max_steering_angle>
+      <topic>/cmd_vel</topic>
+      <odom_topic>odom</odom_topic>
+      <tf_topic>tf</tf_topic>
+      <frame_id>odom</frame_id>
+      <child_frame_id>base_footprint</child_frame_id>
+    </plugin>
+    <plugin
+      filename="ignition-gazebo-joint-state-publisher-system"
+      name="ignition::gazebo::systems::JointStatePublisher">
+    </plugin>
+    <plugin
+      filename="ignition-gazebo-imu-system"
+      name="ignition::gazebo::systems::Imu">
+    </plugin>
+  </gazebo>
 </robot>

File: urdf/imu.urdf.xacro (robot description, xacro)
@@ -2,19 +2,23 @@
 <robot name="imu" xmlns:xacro="http://ros.org/wiki/xacro">
   <xacro:property name="M_PI" value="3.1415926535897931"/>
-  <link
-    name="imu_link">
+  <link name="imu_link">
+    <inertial>
+      <mass value="0.001"/>
+      <inertia ixx="0.0001" ixy="0" ixz="0" iyy="0.0001" iyz="0" izz="0.0001"/>
+    </inertial>
   </link>
-  <joint
-    name="imu_joint"
-    type="fixed">
-    <origin
-      xyz="0 0 ${0.025 - 0.0295 + 0.0965/2 + 0.0678410821576746}"
-      rpy="0 0 ${-M_PI/2}" />
-    <parent
-      link="base_link" />
-    <child
-      link="imu_link" />
-    <axis
-      xyz="0 0 0" />
+  <joint name="imu_joint" type="fixed">
+    <origin xyz="0 0 0.11" rpy="0 0 ${-M_PI/2}" />
+    <parent link="base_link" />
+    <child link="imu_link" />
   </joint>
+  <gazebo reference="imu_link">
+    <sensor name="imu_sensor" type="imu">
+      <always_on>1</always_on>
+      <update_rate>50</update_rate>
+      <visualize>false</visualize>
+      <topic>imu</topic>
+      <gz_frame_id>imu_link</gz_frame_id>
+    </sensor>
+  </gazebo>
 </robot>

File: urdf/mentorpi.xacro (robot description, xacro)
@@ -1,5 +1,4 @@
 <?xml version="1.0" encoding="utf-8"?>
 <robot name="rosmentor" xmlns:xacro="http://ros.org/wiki/xacro">
-    <xacro:property name="machine"      value="$(env MACHINE_TYPE)"/>
     <xacro:include filename="$(find mentorpia1_simulator)/urdf/ackerman.xacro"/>
     <xacro:include filename="$(find mentorpia1_simulator)/urdf/inertial_matrix.xacro" />
